Commit message: import_vel_controller

File: scara_description/urdf/scara.xacro (robot description, xacro)
@@ -63,5 +63,5 @@
     <limit effort="1000.0" lower="-1.57" upper="1.57" velocity="0.5"/>
     <axis xyz = "0 0 1"/>
-    <dynamics damping="0.2" friction="0.6" />
+    <dynamics damping="0.2" friction="0.1" />
   </joint>
   <!-- link 1 -->
@@ -120,5 +120,5 @@
     <limit effort="1000.0" lower="-1.57" upper="1.57" velocity="0.5"/>
     <axis xyz = "0 0 1"/>
-    <dynamics damping="0.2" friction="0.6" />
+    <dynamics damping="0.2" friction="0.1" />
   </joint>
   <!-- link 2 -->
@@ -161,5 +161,5 @@
       <mass value="0.5" />
       <origin xyz="0 0 0" rpy="0 0 0" />
-      v<inertia ixx="0.5" ixy="0" ixz="0" iyy="0.5" iyz="0" izz="0.5" />
+      <inertia ixx="0.5" ixy="0" ixz="0" iyy="0.5" iyz="0" izz="0.5" />
     </inertial>
     <collision>

Commit message: change friction

File: scara_description/urdf/scara.xacro (robot description, xacro)
@@ -47,5 +47,5 @@
       <mass value="0.5" />
       <origin xyz="0 0 0.05" rpy="0 0 0" />
-      v<inertia ixx="0.5" ixy="0" ixz="0" iyy="0.5" iyz="0" izz="0.5" />
+      <inertia ixx="0.5" ixy="0" ixz="0" iyy="0.5" iyz="0" izz="0.5" />
     </inertial>
     <collision>
@@ -63,5 +63,5 @@
     <limit effort="1000.0" lower="-1.57" upper="1.57" velocity="0.5"/>
     <axis xyz = "0 0 1"/>
-    <dynamics damping="0.2" friction="0.1" />
+    <dynamics damping="0.2" friction="0.5" />
   </joint>
   <!-- link 1 -->
@@ -120,5 +120,5 @@
     <limit effort="1000.0" lower="-1.57" upper="1.57" velocity="0.5"/>
     <axis xyz = "0 0 1"/>
-    <dynamics damping="0.2" friction="0.1" />
+    <dynamics damping="0.2" friction="0.5" />
   </joint>
   <!-- link 2 -->

Commit message: update pid value

File: scara_description/urdf/scara.xacro (robot description, xacro)
@@ -63,5 +63,5 @@
     <limit effort="1000.0" lower="-1.57" upper="1.57" velocity="0.5"/>
     <axis xyz = "0 0 1"/>
-    <dynamics damping="0.2" friction="0.5" />
+    <dynamics damping="0.2" friction="0.1" />
   </joint>
   <!-- link 1 -->
@@ -120,5 +120,5 @@
     <limit effort="1000.0" lower="-1.57" upper="1.57" velocity="0.5"/>
     <axis xyz = "0 0 1"/>
-    <dynamics damping="0.2" friction="0.5" />
+    <dynamics damping="0.2" friction="0.1" />
   </joint>
   <!-- link 2 -->
